Commit message: Add chase_moveit.launch
1. Add chase_moveit.launch
2. Change file name jessi_arm -> jessiarm in moveit folder
3. Change jessi_arm -> jessiarm in launch, xml, text files

File: jessiarm_description/urdf/jessiarm.xacro (robot description, xacro)
@@ -13,5 +13,5 @@
           <origin xyz="0 0 0" rpy="0 0 0"/>
           <geometry>
-              <mesh filename="package://jessi_arm_description/meshes/base_link.stl" scale="0.001 0.001 0.001"/>
+              <mesh filename="package://jessiarm_description/meshes/base_link.stl" scale="0.001 0.001 0.001"/>
           </geometry>
       </collision>
@@ -19,5 +19,5 @@
           <origin xyz="0 0 0" rpy="0 0 0"/>
           <geometry>
-              <mesh filename="package://jessi_arm_description/meshes/base_link.stl" scale="0.001 0.001 0.001"/>
+              <mesh filename="package://jessiarm_description/meshes/base_link.stl" scale="0.001 0.001 0.001"/>
           </geometry>
           <material name="black"/>
@@ -42,5 +42,5 @@
       <origin xyz="0 0 0" rpy="0 0 0"/>
       <geometry>
-        <mesh filename="package://jessi_arm_description/meshes/link1.stl" scale="0.001 0.001 0.001"/>
+        <mesh filename="package://jessiarm_description/meshes/link1.stl" scale="0.001 0.001 0.001"/>
       </geometry>
       <material name="blue"/>
@@ -49,5 +49,5 @@
       <origin xyz="0 0 0" rpy="0 0 0"/>
       <geometry>
-        <mesh filename="package://jessi_arm_description/meshes/link1.stl" scale="0.001 0.001 0.001"/>
+        <mesh filename="package://jessiarm_description/meshes/link1.stl" scale="0.001 0.001 0.001"/>
       </geometry>
     </collision>
@@ -71,5 +71,5 @@
       <origin xyz="0 0 0" rpy="0 0 0"/>
       <geometry>
-        <mesh filename="package://jessi_arm_description/meshes/link2.stl" scale="0.001 0.001 0.001"/>
+        <mesh filename="package://jessiarm_description/meshes/link2.stl" scale="0.001 0.001 0.001"/>
       </geometry>
       <material name="green"/>
@@ -78,5 +78,5 @@
       <origin xyz="0 0 0.0019" rpy="0 0 0"/>
       <geometry>
-        <mesh filename="package://jessi_arm_description/meshes/link2.stl" scale="0.001 0.001 0.001"/>
+        <mesh filename="package://jessiarm_description/meshes/link2.stl" scale="0.001 0.001 0.001"/>
       </geometry>
     </collision>
@@ -100,5 +100,5 @@
       <origin xyz="0 0 0" rpy="0 0 0"/>
       <geometry>
-        <mesh filename="package://jessi_arm_description/meshes/link3.stl" scale="0.001 0.001 0.001"/>
+        <mesh filename="package://jessiarm_description/meshes/link3.stl" scale="0.001 0.001 0.001"/>
       </geometry>
       <material name="orange"/>
@@ -107,5 +107,5 @@
       <origin xyz="0 0 0" rpy="0 0 0"/>
       <geometry>
-        <mesh filename="package://jessi_arm_description/meshes/link3.stl" scale="0.001 0.001 0.001"/>
+        <mesh filename="package://jessiarm_description/meshes/link3.stl" scale="0.001 0.001 0.001"/>
       </geometry>
     </collision>
@@ -129,5 +129,5 @@
       <origin xyz="0 0 0" rpy="0 0 0"/>
       <geometry>
-        <mesh filename="package://jessi_arm_description/meshes/link4.stl" scale="0.001 0.001 0.001"/>
+        <mesh filename="package://jessiarm_description/meshes/link4.stl" scale="0.001 0.001 0.001"/>
       </geometry>
       <material name="red"/>
@@ -136,5 +136,5 @@
       <origin xyz="0 0 0" rpy="0 0 0"/>
       <geometry>
-        <mesh filename="package://jessi_arm_description/meshes/link4.stl" scale="0.001 0.001 0.001"/>
+        <mesh filename="package://jessiarm_description/meshes/link4.stl" scale="0.001 0.001 0.001"/>
       </geometry>
     </collision>
@@ -158,5 +158,5 @@
       <origin xyz="0 0 0" rpy="0 0 0"/>
       <geometry>
-        <mesh filename="package://jessi_arm_description/meshes/link5.stl" scale="0.001 0.001 0.001"/>
+        <mesh filename="package://jessiarm_description/meshes/link5.stl" scale="0.001 0.001 0.001"/>
       </geometry>
       <material name="white"/>
@@ -165,5 +165,5 @@
       <origin xyz="0 0 0" rpy="0 0 0"/>
       <geometry>
-        <mesh filename="package://jessi_arm_description/meshes/link5.stl" scale="0.001 0.001 0.001"/>
+        <mesh filename="package://jessiarm_description/meshes/link5.stl" scale="0.001 0.001 0.001"/>
       </geometry>
     </collision>

File: jessiarm_description/urdf/jessiarm_robot.xacro (robot description, xacro)
@@ -1,13 +1,13 @@
 <?xml version="1.0"?>
 <!-- Jessi Arm Chain -->
-<robot name="jessi_arm" xmlns:xacro="http://ros.org/wiki/xacro">
+<robot name="jessiarm" xmlns:xacro="http://ros.org/wiki/xacro">
   <!-- Import Rviz colors -->
-  <xacro:include filename="$(find jessi_arm_description)/urdf/materials.xacro" />
+  <xacro:include filename="$(find jessiarm_description)/urdf/materials.xacro" />
   <!-- Import all Gazebo-customization elements, including Gazebo colors -->
-  <!-- <xacro:include filename="$(find jessi_arm_description)/urdf/jessi_arm.gazebo.xacro" /> -->
+  <!-- <xacro:include filename="$(find jessiarm_description)/urdf/jessiarm.gazebo.xacro" /> -->
   <!-- Import Transmission -->
-  <!-- <xacro:include filename="$(find jessi_arm_description)/urdf/jessi_arm.transmission.xacro" /> -->
+  <!-- <xacro:include filename="$(find jessiarm_description)/urdf/jessiarm.transmission.xacro" /> -->
   <!-- Import URDF -->
-  <xacro:include filename="$(find jessi_arm_description)/urdf/jessi_arm.xacro" />
+  <xacro:include filename="$(find jessiarm_description)/urdf/jessiarm.xacro" />
   <!-- World -->
   <link name="world"/>
